File: electronics/control-pendant-v1.kicad_sch (KiCad schematic)
At the start: 63 parts, among them J1 22-28-4034, J18 M20-7821042, J2 22-28-4034, J3 22-28-4034, J4 1727010, J5 22-28-4034, J6 USB_C_Receptacle_USB2.0, J7 22-28-4034, Q1 MMSS8050-H-TP, Q2 MMSS8050-H-TP, Q3 SQ2361AEES-T1_GE3, Q4 SQ2361AEES-T1_GE3, U1 CP2102N-A02-GQFN24R, U2 ESP32-S3-WROOM-1-N8R8, U4 LT8619, U5 BX0033

Commit message: 05/01/2025 Final Commit
Other:
- company: Tribonix  -> (none)
- title: Control Electronics for GDIP V1 -> Control Electronics for GDIP
Changed lines of the file:
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@@
 	(paper "A3")
 	(title_block
-		(title "Control Electronics for GDIP V1")
-		(date "2024-11-26")
-		(company "Tribonix ")
+		(title "Control Electronics for GDIP")
+		(date "2025-01-05")
+		(rev "v1.0")
 		(comment 1 "Drawn By: Filip Hanus")
 	)
